Commit message: Update model

File: model/description/ros2_control.xacro (robot description, xacro)
@@ -2,5 +2,53 @@
 <robot xmlns:xacro="http://www.ros.org/wiki/xacro" name="robot">
     <xacro:unless value="$(arg sim_mode)">
-        <!-- Real Robot Configuration  -->
+        <ros2_control name="SentinelHardwareInterface" type="system">
+            <hardware>
+                <plugin>sentinel_hardware_interface/SentinelHardwareInterface</plugin>
+                <param name="left_front_wheel">left_front_wheel_joint</param>
+                <param name="left_rear_wheel">left_rear_wheel_joint</param>
+                <param name="right_front_wheel">right_front_wheel_joint</param>
+                <param name="right_rear_wheel">right_rear_wheel_joint</param>
+                <param name="device">/dev/ttyUSB0</param>
+                <param name="timeout_ms">1000</param>
+                <param name="loop_rate">30</param>
+                <param name="count_per_rev">20</param>
+                <param name="kp">100</param>
+                <param name="kd">30</param>
+                <param name="ki">10</param>
+                <param name="ko">100</param>
+            </hardware>
+            <joint name="left_front_wheel_joint">
+                <command_interface name="velocity">
+                    <param name="min">-10</param>
+                    <param name="max">10</param>
+                </command_interface>
+                <state_interface name="position" />
+                <state_interface name="velocity" />
+            </joint>
+            <joint name="left_rear_wheel_joint">
+                <command_interface name="velocity">
+                    <param name="min">-10</param>
+                    <param name="max">10</param>
+                </command_interface>
+                <state_interface name="position" />
+                <state_interface name="velocity" />
+            </joint>
+            <joint name="right_front_wheel_joint">
+                <command_interface name="velocity">
+                    <param name="min">-10</param>
+                    <param name="max">10</param>
+                </command_interface>
+                <state_interface name="position" />
+                <state_interface name="velocity" />
+            </joint>
+            <joint name="right_rear_wheel_joint">
+                <command_interface name="velocity">
+                    <param name="min">-10</param>
+                    <param name="max">10</param>
+                </command_interface>
+                <state_interface name="position" />
+                <state_interface name="velocity" />
+            </joint>
+        </ros2_control>
     </xacro:unless>
     <xacro:if value="$(arg sim_mode)">
