Commit message: Add new model

File: model/description/camera.xacro (robot description, xacro)
@@ -6,7 +6,7 @@
     <!-- Body & Camera Joint !-->
     <joint name="camera_joint" type="fixed">
-        <parent link="base_link" />
+        <parent link="chassis_mid" />
         <child link="camera_link" />
-        <origin xyz="0.1 0 0.19" rpy="0 0 0" />
+        <origin xyz="${chassis_total_length/2 - 0.007 - 0.005} 0 ${0.02}" rpy="0 0 0" />
     </joint>
     <!-- Camera !-->

File: model/description/lidar.xacro (robot description, xacro)
@@ -24,7 +24,9 @@
     <!-- Body & Lidar Joint !-->
     <joint name="lidar_joint" type="fixed">
-        <parent link="base_link" />
+        <parent link="chassis_mid" />
         <child link="lidar" />
-        <origin xyz="-0.04 -0.04 0.215" rpy="0.0 0.0 0.0" />
+        <origin
+            xyz="-${chassis_total_length/2 - 0.0295 - 0.045} -${chassis_small_width/2 - 0.0295 - 0.02} ${0.026 *2}"
+            rpy="0.0 0.0 0.0" />
     </joint>
     <gazebo reference="lidar">

File: model/description/others.xacro (robot description, xacro)
@@ -6,9 +6,208 @@
     <!-- =================================================================================== -->
     <!-- Motor -->
-    <xacro:macro name="motor" params="prefix">
+    <xacro:macro name="motors" params="prefix">
         <link name="${prefix}_motor">
             <visual>
                 <geometry>
-                    <box size="0.064 0.019 0.021" />
+                    <cylinder radius="${motor_radius}" length="${motor_length}" />
+                </geometry>
+                <origin xyz="0.0 0.0 0.0" rpy="0 0 0" />
+                <material name="Gray" />
+            </visual>
+            <collision>
+                <geometry>
+                    <cylinder radius="${motor_radius}" length="${motor_length}" />
+                </geometry>
+            </collision>
+            <xacro:inertial_cylinder mass="${motor_mass}" length="${motor_length}"
+                radius="${motor_radius}">
+                <origin xyz="0.0 0.0 0.0" rpy="0 0 0" />
+            </xacro:inertial_cylinder>
+        </link>
+    </xacro:macro>
+    <xacro:motors prefix="left_front" />
+    <xacro:motors prefix="left_rear" />
+    <xacro:motors prefix="right_front" />
+    <xacro:motors prefix="right_rear" />
+    <joint name="left_front_motor_joint" type="fixed">
+        <parent link="left_front_wheel" />
+        <child link="left_front_motor" />
+        <origin xyz="0.0 0.0 -${motor_length/2 + wheel_thickness/2}" rpy="0 0 0" />
+        <axis xyz="0 0 1" />
+    </joint>
+    <joint name="left_rear_motor_joint" type="fixed">
+        <parent link="left_rear_wheel" />
+        <child link="left_rear_motor" />
+        <origin xyz="0.0 0.0 -${motor_length/2 + wheel_thickness/2}" rpy="0 0 0" />
+        <axis xyz="0 0 1" />
+    </joint>
+    <joint name="right_front_motor_joint" type="fixed">
+        <parent link="right_front_wheel" />
+        <child link="right_front_motor" />
+        <origin xyz="0.0 0.0 -${motor_length/2 + wheel_thickness/2}" rpy="0 0 0" />
+        <axis xyz="0 0 1" />
+    </joint>
+    <joint name="right_rear_motor_joint" type="fixed">
+        <parent link="right_rear_wheel" />
+        <child link="right_rear_motor" />
+        <origin xyz="0.0 0.0 -${motor_length/2 + wheel_thickness/2}" rpy="0 0 0" />
+        <axis xyz="0 0 1" />
+    </joint>
+    <!-- =================================================================================== -->
+    <!-- |                                    Arduino                                      | -->
+    <!-- =================================================================================== -->
+    <!-- Raspberry -->
+    <link name="arduino">
+        <visual>
+            <geometry>
+                <box size="0.082 0.053 0.007" />
+            </geometry>
+            <origin xyz="0.0 0.0 0.0" rpy="0.0 0.0 0.0" />
+        </visual>
+        <collision>
+            <geometry>
+                <box size="0.082 0.053 0.007" />
+            </geometry>
+        </collision>
+        <xacro:inertial_box mass="0.080" x="0.082" y="0.053" z="0.007">
+            <origin xyz="0 0 0" rpy="0 0 0" />
+        </xacro:inertial_box>
+    </link>
+    <!-- Arduino joint-->
+    <joint name="arduino_joint" type="fixed">
+        <parent link="chassis_bottom" />
+        <child link="arduino" />
+        <origin
+            xyz="-${chassis_total_length/2 - 0.0265 - 0.03} ${chassis_small_width/2 - 0.041 - 0.015} ${0.0035 + chassis_height} "
+            rpy="0 0.0 ${pi/2}" />
+    </joint>
+    <!-- =================================================================================== -->
+    <!-- |                                  Battery                                        | -->
+    <!-- =================================================================================== -->
+    <!-- Battery -->
+    <link name="battery">
+        <visual>
+            <geometry>
+                <box size="0.075 0.065 0.035" />
+            </geometry>
+            <origin xyz="0.0 0.0 0.0" rpy="0.0 0.0 0.0" />
+            <material name="Red" />
+        </visual>
+        <collision>
+            <geometry>
+                <box size="0.071 0.065 0.035" />
+            </geometry>
+        </collision>
+        <xacro:inertial_box mass="0.385" x="0.071" y="0.065" z="0.035">
+            <origin xyz="0 0 0" rpy="0 0 0" />
+        </xacro:inertial_box>
+    </link>
+    <!-- Battery Mid Joint!-->
+    <joint name="battery_mid_joint" type="fixed">
+        <parent link="chassis_bottom" />
+        <child link="battery" />
+        <origin
+            xyz="-${chassis_total_length/2 - 0.0325 - 0.035} -${chassis_small_width/2 - 0.0375 - 0.015} ${0.0175 + chassis_height}"
+            rpy="0.0 0.0 ${pi/2}" />
+    </joint>
+    <!-- =================================================================================== -->
+    <!-- |                                  PowerBank                                      | -->
+    <!-- =================================================================================== -->
+    <!-- PowerBank -->
+    <link name="powerbank">
+        <visual>
+            <geometry>
+                <box size="0.143 0.070 0.025" />
+            </geometry>
+            <origin xyz="0.0 0.0 0.0" rpy="0.0 0.0 0.0" />
+            <material name="White" />
+        </visual>
+        <collision>
+            <geometry>
+                <box size="0.143 0.070 0.025" />
+            </geometry>
+        </collision>
+        <xacro:inertial_box mass="0.395" x="0.143" y="0.070" z="0.025">
+            <origin xyz="0 0 0" rpy="0 0 0" />
+        </xacro:inertial_box>
+    </link>
+    <!-- powerbank joint-->
+    <joint name="powerbank_joint" type="fixed">
+        <parent link="chassis_mid" />
+        <child link="powerbank" />
+        <origin
+            xyz="${chassis_total_length/2 - 0.0715 - 0.025} ${chassis_small_width/2 - 0.035 - 0.015} ${chassis_height + 0.0125}"
+            rpy="0.0 0.0 0.0" />
+    </joint>
+    <!-- =================================================================================== -->
+    <!-- |                               Motor Driver                                      | -->
+    <!-- =================================================================================== -->
+    <!-- Motor Driver -->
+    <link name="motor_driver">
+        <visual>
+            <geometry>
+                <box size="0.044 0.044 0.02" />
+            </geometry>
+            <origin xyz="0.0 0.0 0.0" rpy="0.0 0.0 0.0" />
+            <material name="Red" />
+        </visual>
+        <collision>
+            <geometry>
+                <box size="0.044 0.044 0.02" />
+            </geometry>
+        </collision>
+        <xacro:inertial_box mass="0.024" x="0.044" y="0.044" z="0.02">
+            <origin xyz="0 0 0" rpy="0 0 0" />
+        </xacro:inertial_box>
+    </link>
+    <!-- Motor Driver Joint-->
+    <joint name="motor_driver_joint" type="fixed">
+        <parent link="chassis_bottom" />
+        <child link="motor_driver" />
+        <origin xyz="0 0 0" rpy="0.0 0.0 0.0" />
+        <origin
+            xyz="${chassis_total_length/2 - 0.022 - 0.01} -${chassis_big_width/2 - 0.022- 0.05} 0.013"
+            rpy="0.0 0.0
+        0.0" />
+    </joint>
+    <!-- =================================================================================== -->
+    <!-- |                                  Raspberry                                      | -->
+    <!-- =================================================================================== -->
+    <!-- Raspberry -->
+    <link name="raspberry_pi">
+        <visual>
+            <geometry>
+                <box size="0.095 0.064 0.025" />
+            </geometry>
+            <origin xyz="0.0 0.0 0.0" rpy="0.0 0.0 0.0" />
+            <material name="DarkGreen" />
+        </visual>
+        <collision>
+            <geometry>
+                <box size="0.095 0.064 0.025" />
+            </geometry>
+        </collision>
+        <xacro:inertial_box mass="0.140" x="0.095" y="0.064" z="0.025">
+            <origin xyz="0 0 0" rpy="0 0 0" />
+        </xacro:inertial_box>
+    </link>
+    <!-- Raspberry joint-->
+    <joint name="raspberry_pi_joint" type="fixed">
+        <parent link="chassis_bottom" />
+        <child link="raspberry_pi" />
+        <origin
+            xyz="${chassis_total_length/2 - 0.04745 -0.03} ${chassis_small_width/2 - 0.032 - 0.015} ${0.0125 + chassis_height}"
+            rpy="0.0 0.0 0.0" />
+    </joint>
+    <!-- =================================================================================== -->
+    <!-- |                               Small Cylinder                                    | -->
+    <!-- =================================================================================== -->
+    <!-- Small_cylinder Macro !-->
+    <xacro:macro
+        name="small_cylinder" params="prefix">
+        <link name="small_cylinder_${prefix}">
+            <visual>
+                <geometry>
+                    <cylinder radius="0.002" length="${small_cylinder_length}" />
                 </geometry>
                 <origin xyz="0.0 0.0 0.0" rpy="0.0 0.0 0.0" />
@@ -17,302 +216,46 @@
             <collision>
                 <geometry>
-                    <box size="0.064 0.019 0.021" />
+                    <cylinder radius="0.002" length="${small_cylinder_length}" />
                 </geometry>
             </collision>
-        </link>
-    </xacro:macro>
-    <!-- Left Front Motor !-->
-    <xacro:motor prefix="left_front" />
-    <!-- Left Rear Motor !-->
-    <xacro:motor prefix="left_rear" />
-    <!-- Right Front Motor !-->
-    <xacro:motor prefix="right_front" />
-    <!-- Right Rear Motor !-->
-    <xacro:motor prefix="right_rear" />
-    <!-- Left Front Motor Joint!-->
-    <joint name="left_front_motor_joint" type="fixed">
-        <parent link="base_link" />
-        <child link="left_front_motor" />
-        <origin xyz="0.0365 0.0390 0.035" rpy="0.0 0.0 0.0" />
-        <xacro:inertial_box mass="0.025" x="0.0365" y="0.0390" z="0.035">
-            <origin xyz="0 0 0" rpy="0 0 0" />
-        </xacro:inertial_box>
-    </joint>
-    <!-- Left Rear Motor Joint!-->
-    <joint name="left_rear_motor_joint" type="fixed">
-        <parent link="base_link" />
-        <child link="left_rear_motor" />
-        <origin xyz="-0.0365 0.039 0.035" rpy="0 0 0" />
-        <xacro:inertial_box mass="0.025" x="-0.0365" y="0.0390" z="0.035">
-            <origin xyz="0 0 0" rpy="0 0 0" />
-        </xacro:inertial_box>
-    </joint>
-    <!-- Right Front Motor Joint!-->
-    <joint name="right_front_motor_joint" type="fixed">
-        <parent link="base_link" />
-        <child link="right_front_motor" />
-        <origin xyz="0.0365 -0.039 0.035" rpy="0 0 0" />
-        <xacro:inertial_box mass="0.025" x="0.0365" y="-0.0390" z="0.035">
-            <origin xyz="0 0 0" rpy="0 0 0" />
-        </xacro:inertial_box>
-    </joint>
-    <!-- Right Rear Motor Joint!-->
-    <joint name="right_rear_motor_joint" type="fixed">
-        <parent link="base_link" />
-        <child link="right_rear_motor" />
-        <origin xyz="-0.0365 -0.039 0.035" rpy="0 0 0" />
-        <xacro:inertial_box mass="0.025" x="-0.0365" y="-0.0390" z="0.035">
-            <origin xyz="0 0 0" rpy="0 0 0" />
-        </xacro:inertial_box>
-    </joint>
-    <!-- =================================================================================== -->
-    <!-- |                                  Battery                                        | -->
-    <!-- =================================================================================== -->
-    <!-- Battery -->
-    <link name="battery">
-        <visual>
-            <geometry>
-                <box size="0.075 0.065 0.035" />
-            </geometry>
-            <origin xyz="0.0 0.0 0.0" rpy="0.0 0.0 0.0" />
-            <material name="NavyBlue" />
-        </visual>
-        <collision>
-            <geometry>
-                <box size="0.071 0.065 0.035" />
-            </geometry>
-        </collision>
-        <xacro:inertial_box mass="0.385" x="0.071" y="0.065" z="0.035">
-            <origin xyz="0 0 0" rpy="0 0 0" />
-        </xacro:inertial_box>
-    </link>
-    <!-- Battery Mid Joint!-->
-    <joint name="battery_mid_joint" type="fixed">
-        <parent link="base_link" />
-        <child link="battery" />
-        <origin xyz="-0.0455 0.0 0.0895" rpy="0.0 0.0 0.0" />
-    </joint>
-    <!-- =================================================================================== -->
-    <!-- |                                  PowerBank                                      | -->
-    <!-- =================================================================================== -->
-    <!-- PowerBank -->
-    <link name="powerbank">
-        <visual>
-            <geometry>
-                <box size="0.143 0.070 0.025" />
-            </geometry>
-            <origin xyz="0.0 0.0 0.0" rpy="0.0 0.0 0.0" />
-            <material name="BlackWheel" />
-        </visual>
-        <collision>
-            <geometry>
-                <box size="0.143 0.070 0.025" />
-            </geometry>
-        </collision>
-        <xacro:inertial_box mass="0.395" x="0.143" y="0.070" z="0.025">
-            <origin xyz="0 0 0" rpy="0 0 0" />
-        </xacro:inertial_box>
-    </link>
-    <!-- Base-powerbank joint-->
-    <joint name="base_powerbank" type="fixed">
-        <parent link="base_link" />
-        <child link="powerbank" />
-        <origin xyz="0.000 0.000 0.0595" rpy="0.0 0.0 0.0" />
-    </joint>
-    <!-- =================================================================================== -->
-    <!-- |                               Motor Driver                                      | -->
-    <!-- =================================================================================== -->
-    <!-- Motor Driver -->
-    <link name="motor_driver">
-        <visual>
-            <geometry>
-                <box size="0.044 0.044 0.02" />
-            </geometry>
-            <origin xyz="0.0 0.0 0.0" rpy="0.0 0.0 0.0" />
-            <material name="Red" />
-        </visual>
-        <collision>
-            <geometry>
-                <box size="0.044 0.044 0.02" />
-            </geometry>
-        </collision>
-        <xacro:inertial_box mass="0.024" x="0.044" y="0.044" z="0.02">
-            <origin xyz="0 0 0" rpy="0 0 0" />
-        </xacro:inertial_box>
-    </link>
-    <!-- Motor Driver Joint-->
-    <joint name="motor_driver_joint" type="fixed">
-        <parent link="base_link" />
-        <child link="motor_driver" />
-        <origin xyz="0.10 0.00 0.060" rpy="0.0 0.0 0.0" />
-    </joint>
-    <!-- =================================================================================== -->
-    <!-- |                                  Raspberry                                      | -->
-    <!-- =================================================================================== -->
-    <!-- Raspberry -->
-    <link name="raspberry">
-        <visual>
-            <geometry>
-                <box size="0.095 0.064 0.025" />
-            </geometry>
-            <origin xyz="0.0 0.0 0.0" rpy="0.0 0.0 0.0" />
-            <material name="DarkGreen" />
-        </visual>
-        <collision>
-            <geometry>
-                <box size="0.095 0.064 0.025" />
-            </geometry>
-        </collision>
-        <xacro:inertial_box mass="0.140" x="0.095" y="0.064" z="0.025">
-            <origin xyz="0 0 0" rpy="0 0 0" />
-        </xacro:inertial_box>
-    </link>
-    <!-- Base-raspberry joint-->
-    <joint name="base_raspberry" type="fixed">
-        <parent link="base_link" />
-        <child link="raspberry" />
-        <origin xyz="0.0455 0.00 0.0845" rpy="0.0 0.0 0.0" />
-    </joint>
-    <!-- =================================================================================== -->
-    <!-- |                               Small Cylinder                                    | -->
-    <!-- =================================================================================== -->
-    <!-- Small_cylinder Macro !-->
-    <xacro:macro name="small_cylinder" params="prefix">
-        <link name="base_mid_${prefix}">
-            <visual>
-                <geometry>
-                    <cylinder radius="0.002" length="0.029" />
-                </geometry>
-                <origin xyz="0.0 0.0 0.0" rpy="0.0 0.0 0.0" />
-                <material name="DarkGold" />
-            </visual>
-            <collision>
-                <geometry>
-                    <cylinder radius="0.002" length="0.029" />
-                </geometry>
-            </collision>
-            <xacro:inertial_cylinder mass="0.001" length="0.029" radius="0.002">
+            <xacro:inertial_cylinder mass="0.001" length="${small_cylinder_length}" radius="0.002">
                 <origin xyz="0 0 0" rpy="0 0 0" />
             </xacro:inertial_cylinder>
         </link>
     </xacro:macro>
-    <!-- Cylinder base-mid left front!-->
-    <xacro:small_cylinder prefix="left_front" />
-    <!-- Cylinder base-mid left front2!-->
-    <xacro:small_cylinder prefix="left_front_2" />
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
File: model/description/robot.urdf.xacro (robot description, xacro)
@@ -5,4 +5,5 @@
     <xacro:arg name="sim_mode" default="false" />
     <xacro:include filename="robot_core.xacro" />
+    <xacro:include filename="wheels.xacro" />
     <xacro:include filename="others.xacro" />
     <xacro:include filename="wheels.xacro" />
