Commit message: Add new model

File: model/description/robot_core.xacro (robot description, xacro)
@@ -39,4 +39,21 @@
     <link name="base_footprint">
     </link>
+    <xacro:property name="chassis_total_length" value="0.25" />
+    <xacro:property name="chassis_small_length" value="0.032" />
+    <xacro:property name="chassis_big_length" value="0.077" />
+    <xacro:property name="chassis_small_width" value="0.2" />
+    <xacro:property name="chassis_big_width" value="0.248" />
+    <xacro:property name="chassis_height" value="0.004" />
+    <xacro:property name="chassis_mass" value="0.240" />
+    <xacro:property name="wheel_radius" value="0.033" />
+    <xacro:property name="wheel_thickness" value="0.026" />
+    <xacro:property name="wheel_mass" value="0.05" />
+    <xacro:property name="wheel_offset_x" value="0.01" />
+    <xacro:property name="wheel_offset_z" value="0.01" />
+    <xacro:property name="motor_radius" value="0.0244" />
+    <xacro:property name="motor_length" value="0.059" />
+    <xacro:property name="motor_mass" value="0.096" />
+    <xacro:property name="motor_bracket_offset" value="0.01" />
+    <xacro:property name="small_cylinder_length" value="0.0435" />
     <!-- =================================================================================== -->
     <!-- |                                    Chassis                                      | -->
@@ -47,95 +64,108 @@
             <visual>
                 <geometry>
-                    <box size="0.032 0.148 0.003" />
+                    <box size="${chassis_small_length} ${chassis_big_width} ${chassis_height}" />
                 </geometry>
-                <origin xyz="-0.111 0 0.02" rpy="0.0 0.0 0.0" />
+                <origin
+                    xyz="${(chassis_small_length + 0.0015 + chassis_big_length)} 0 0"
+                    rpy="0.0 0.0 0.0" />
                 <material name="WoodYellow" />
             </visual>
             <visual>
                 <geometry>
-                    <box size="0.077 0.1 0.003" />
+                    <box size="${chassis_big_length} ${chassis_small_width} ${chassis_height}" />
                 </geometry>
-                <origin xyz="-0.056 0 0.02" rpy="0.0 0.0 0.0" />
+                <origin xyz="${chassis_big_length/2+(chassis_small_length+0.003)/2} 0 0"
+                    rpy="0.0 0.0 0.0" />
                 <material name="WoodYellow" />
             </visual>
             <visual>
                 <geometry>
-                    <box size="0.035 0.148 0.003" />
+                    <box
+                        size="${chassis_small_length + 0.003} ${chassis_big_width} ${chassis_height}" />
                 </geometry>
-                <origin xyz="0 0 0.02" rpy="0.0 0.0 0.0" />
+                <origin xyz="0 0 0" rpy="0.0 0.0 0.0" />
                 <material name="WoodYellow" />
             </visual>
             <visual>
                 <geometry>
-                    <box size="0.077 0.1 0.003" />
+                    <box size="${chassis_big_length} ${chassis_small_width} ${chassis_height}" />
                 </geometry>
-                <origin xyz="0.056 0 0.02" rpy="0.0 0.0 0.0" />
+                <origin xyz="-${chassis_big_length/2+(chassis_small_length+0.003)/2} 0 0"
+                    rpy="0.0 0.0 0.0" />
                 <material name="WoodYellow" />
             </visual>
             <visual>
                 <geometry>
-                    <box size="0.032 0.148 0.003" />
+                    <box size="${chassis_small_length} ${chassis_big_width} ${chassis_height}" />
                 </geometry>
-                <origin xyz="0.111 0 0.02" rpy="0.0 0.0 0.0" />
+                <origin
+                    xyz="-${(chassis_small_length + 0.0015 + chassis_big_length)} 0 0"
+                    rpy="0.0 0.0 0.0" />
                 <material name="WoodYellow" />
             </visual>
             <collision>
                 <geometry>
-                    <box size="0.032 0.148 0.003" />
+                    <box size="${chassis_small_length} ${chassis_big_width} ${chassis_height}" />
                 </geometry>
-                <origin xyz="-0.111 0 0.02" rpy="0.0 0.0 0.0" />
+                <origin
+                    xyz="${(chassis_small_length + 0.0015 + chassis_big_length)} 0 0"
+                    rpy="0.0 0.0 0.0" />
             </collision>
             <collision>
                 <geometry>
-                    <box size="0.077 0.1 0.003" />
+                    <box size="${chassis_big_length} ${chassis_small_width} ${chassis_height}" />
                 </geometry>
-                <origin xyz="-0.056 0 0.02" rpy="0.0 0.0 0.0" />
+                <origin xyz="${chassis_big_length/2+(chassis_small_length+0.003)/2} 0 0"
+                    rpy="0.0 0.0 0.0" />
             </collision>
             <collision>
                 <geometry>
-                    <box size="0.035 0.148 0.003" />
+                    <box
+                        size="${chassis_small_length + 0.003} ${chassis_big_width} ${chassis_height}" />
                 </geometry>
-                <origin xyz="0 0 0.02" rpy="0.0 0.0 0.0" />
+                <origin xyz="0 0 0" rpy="0.0 0.0 0.0" />
             </collision>
             <collision>
                 <geometry>
-                    <box size="0.077 0.1 0.003" />
+                    <box size="${chassis_big_length} ${chassis_small_width} ${chassis_height}" />
                 </geometry>
-                <origin xyz="0.056 0 0.02" rpy="0.0 0.0 0.0" />
+                <origin xyz="-${chassis_big_length/2+(chassis_small_length+0.003)/2} 0 0"
+                    rpy="0.0 0.0 0.0" />
             </collision>
             <collision>
                 <geometry>
-                    <box size="0.032 0.148 0.003" />
+                    <box size="${chassis_small_length} ${chassis_big_width} ${chassis_height}" />
                 </geometry>
-                <origin xyz="0.111 0 0.02" rpy="0.0 0.0 0.0" />
+                <origin
+                    xyz="-${(chassis_small_length + 0.0015 + chassis_big_length)} 0 0"
+                    rpy="0.0 0.0 0.0" />
             </collision>
-            <xacro:inertial_box mass="0.064" x="0.25" y="0.148" z="0.003">
-                <origin xyz="0 0 0.04" rpy="0 0 0" />
-            </xacro:inertial_box>
+            <xacro:inertial_box mass="${chassis_mass}" x="${chassis_total_length}"
+                y="${chassis_big_width}"
+                z="${chassis_height}">
+                <!--TODO:Check  -->
+                <origin
+                    xyz="${chassis_total_length} ${chassis_big_width} ${chassis_height}"
+                    rpy="0 0 0" />` </xacro:inertial_box>
         </link>
     </xacro:macro>
     <!-- Chassis bottom !-->
-    <xacro:chassis postfix="bottom" />
+    <xacro:chassis
+        postfix="bottom" />
     <!-- Chassis mid !-->
     <xacro:chassis postfix="mid" />
-    <!-- Chassis top !-->
-    <xacro:chassis postfix="top" />
     <!-- Chassis bottom !-->
-    <joint name="chassis_bottom_joint" type="fixed">
+    <joint name="chassis_bottom_joint"
+        type="fixed">
         <parent link="base_link" />
         <child link="chassis_bottom" />
-        <origin xyz="0 0 0" />
+        <origin xyz="0 0 ${wheel_radius - wheel_radius + motor_radius + motor_bracket_offset}" />
     </joint>
     <!-- Chassis mid !-->
-    <joint name="chassis_mid_joint" type="fixed">
-        <parent link="base_link" />
+    <joint
+        name="chassis_mid_joint" type="fixed">
+        <parent link="chassis_bottom" />
         <child link="chassis_mid" />
-        <origin xyz="0.0 0.0 0.028" />
-    </joint>
-    <!-- Chassis top !-->
-    <joint name="chassis_top_joint" type="fixed">
-        <parent link="base_link" />
-        <child link="chassis_top" />
-        <origin xyz="0.00 0.00 0.148" />
+        <origin xyz="0.0 0.0 ${small_cylinder_length + chassis_height}" />
     </joint>
 </robot>

File: model/description/wheels.xacro (robot description, xacro)
@@ -4,107 +4,60 @@
     <!-- |                                     Wheels                                      | -->
     <!-- =================================================================================== -->
-    <!-- Left Front Wheel Joint!-->
+    <xacro:macro name="wheels" params="prefix">
+        <link name="${prefix}_wheel">
+            <visual>
+                <geometry>
+                    <cylinder radius="${wheel_radius}" length="${wheel_thickness}" />
+                </geometry>
+                <origin xyz="0.0 0.0 0.0" rpy="0 0 0" />
+                <material name="BlackWheel" />
+            </visual>
+            <collision>
+                <geometry>
+                    <!-- <cylinder radius=${wheel_radius}" length="${wheel_thickness}" /> -->
+                    <sphere radius="${wheel_radius}" />
+                </geometry>
+            </collision>
+            <xacro:inertial_cylinder mass="${wheel_mass}" length="${wheel_thickness}"
+                radius="${wheel_radius}">
+                <origin xyz="0.0 0.0 0.0" rpy="0 0 0" />
+            </xacro:inertial_cylinder>
+        </link>
+    </xacro:macro>
+    <xacro:wheels prefix="left_front" />
+    <xacro:wheels prefix="left_rear" />
+    <xacro:wheels prefix="right_front" />
+    <xacro:wheels prefix="right_rear" />
     <joint name="left_front_wheel_joint" type="continuous">
         <parent link="base_link" />
         <child link="left_front_wheel" />
-        <origin xyz="0.0575 0.0640 0.035" rpy="${-pi/2} 0.0 0.0" />
+        <origin
+            xyz="${chassis_big_length/2+(chassis_small_length+0.003)/2} ${chassis_small_width/2 + 0.015} 0.0"
+            rpy="${-pi/2} 0.0 0.0" />
         <axis xyz="0 0 1" />
     </joint>
-    <!-- Left Front Wheel !-->
-    <link name="left_front_wheel">
-        <visual>
-            <geometry>
-                <cylinder radius="0.035" length="0.025" />
-            </geometry>
-            <origin xyz="0.0 0.0 0.0" rpy="0 0 0" />
-            <material name="BlackWheel" />
-        </visual>
-        <collision>
-            <geometry>
-                <!-- <cylinder radius="0.0325" length="0.026" /> -->
-                <sphere radius="0.0325" />
-            </geometry>
-        </collision>
-        <xacro:inertial_cylinder mass="0.027" length="0.025" radius="0.035">
-            <origin xyz="0.0 0.0 0.0" rpy="0 0 0" />
-        </xacro:inertial_cylinder>
-    </link>
-    <!-- Right Front Wheel Joint!-->
+    <joint name="left_rear_wheel_joint" type="continuous">
+        <parent link="base_link" />
+        <child link="left_rear_wheel" />
+        <origin
+            xyz="-${chassis_big_length/2+(chassis_small_length+0.003)/2} ${chassis_small_width/2 + 0.015} 0.0"
+            rpy="${-pi/2} 0.0 0.0" />
+        <axis xyz="0 0 1" />
+    </joint>
     <joint name="right_front_wheel_joint" type="continuous">
         <parent link="base_link" />
         <child link="right_front_wheel" />
-        <origin xyz="0.0575 -0.0640 0.035" rpy="${pi/2} 0.0 0.0" />
+        <origin
+            xyz="${chassis_big_length/2+(chassis_small_length+0.003)/2} -${chassis_small_width/2 + 0.015} 0.0"
+            rpy="${pi/2} 0.0 0.0" />
         <axis xyz="0 0 -1" />
     </joint>
-    <!-- Right Front Wheel !-->
-    <link name="right_front_wheel">
-        <visual>
-            <geometry>
-                <cylinder radius="0.035" length="0.025" />
-            </geometry>
-            <origin xyz="0.0 0.0 0.0" rpy="0 0 0" />
-            <material name="BlackWheel" />
-        </visual>
-        <collision>
-            <geometry>
-                <!-- <cylinder radius="0.0325" length="0.026" /> -->
-                <sphere radius="0.0325" />
-            </geometry>
-        </collision>
-        <xacro:inertial_cylinder mass="0.027" length="0.025" radius="0.035">
-            <origin xyz="0.0 0.0 0.0" rpy="0 0 0" />
-        </xacro:inertial_cylinder>
-    </link>
-    <!-- Left Rear Wheel Joint!-->
-    <joint name="left_rear_wheel_joint" type="continuous">
-        <parent link="base_link" />
-        <child link="left_rear_wheel" />
-        <origin xyz="-0.0575 0.0640 0.035" rpy="-${pi/2} 0.0 0.0" />
-        <axis xyz="0 0 1" />
-    </joint>
-    <!-- Left Rear Wheel !-->
-    <link name="left_rear_wheel">
-        <visual>
-            <geometry>
-                <cylinder radius="0.035" length="0.025" />
-            </geometry>
-            <origin xyz="0.0 0.0 0.0" rpy="0 0 0" />
-            <material name="BlackWheel" />
-        </visual>
-        <collision>
-            <geometry>
-                <!-- <cylinder radius="0.0325" length="0.026" /> -->
-                <sphere radius="0.0325" />
-            </geometry>
-        </collision>
-        <xacro:inertial_cylinder mass="0.027" length="0.025" radius="0.035">
-            <origin xyz="0.0 0.0 0.0" rpy="0 0 0" />
-        </xacro:inertial_cylinder>
-    </link>
-    <!-- Right Rear Wheel Joint!-->
     <joint name="right_rear_wheel_joint" type="continuous">
         <parent link="base_link" />
         <child link="right_rear_wheel" />
-        <origin xyz="-0.0575 -0.0640 0.035" rpy="${pi/2} 0.0 0.0" />
+        <origin
+            xyz="-${chassis_big_length/2+(chassis_small_length+0.003)/2} -${chassis_small_width/2 + 0.015} 0.0"
+            rpy="${pi/2} 0.0 0.0" />
         <axis xyz="0 0 -1" />
     </joint>
-    <!-- Right Rear Wheel !-->
-    <link name="right_rear_wheel">
-        <visual>
-            <geometry>
-                <cylinder radius="0.035" length="0.025" />
-            </geometry>
-            <origin xyz="0.0 0.0 0.0" rpy="0 0 0" />
-            <material name="BlackWheel" />
-        </visual>
-        <collision>
-            <geometry>
-                <!-- <cylinder radius="0.0325" length="0.026" /> -->
-                <sphere radius="0.0325" />
-            </geometry>
-        </collision>
-        <xacro:inertial_cylinder mass="0.027" length="0.025" radius="0.035">
-            <origin xyz="0.0 0.0 0.0" rpy="0 0 0" />
-        </xacro:inertial_cylinder>
-    </link>
 </robot>
