Commit message: Update and fix model

File: model/description/others.xacro (robot description, xacro)
@@ -224,9 +224,7 @@
         </link>
     </xacro:macro>
-    <xacro:small_cylinder
-        prefix="left_front" />
+    <xacro:small_cylinder prefix="left_front" />
     <xacro:small_cylinder prefix="right_front" />
-    <xacro:small_cylinder
-        prefix="left_rear" />
+    <xacro:small_cylinder prefix="left_rear" />
     <xacro:small_cylinder prefix="right_rear" />
     <joint

File: model/description/rgbd_camera.xacro (robot description, xacro)
@@ -4,8 +4,9 @@
     <!-- |                                   Camera                                        | -->
     <!-- =================================================================================== -->
+    <!-- Body & Camera Joint !-->
     <joint name="camera_joint" type="fixed">
-        <parent link="chassis_top" />
+        <parent link="chassis_mid" />
         <child link="camera_link" />
-        <origin xyz="0.1 0 0.05" rpy="0 0 0" />
+        <origin xyz="${chassis_total_length/2 - 0.007 - 0.005} 0 ${0.02}" rpy="0 0 0" />
     </joint>
     <!-- Camera !-->

File: model/description/robot.urdf.xacro (robot description, xacro)
@@ -5,5 +5,4 @@
     <xacro:arg name="sim_mode" default="false" />
     <xacro:include filename="robot_core.xacro" />
-    <xacro:include filename="wheels.xacro" />
     <xacro:include filename="others.xacro" />
     <xacro:include filename="wheels.xacro" />

File: model/description/robot_core.xacro (robot description, xacro)
@@ -20,5 +20,5 @@
         <color rgba="1 1 1 1.0" />
     </material>
-    <material name="Grey">
+    <material name="Gray">
         <color rgba="0.7 0.7 0.7 1.0" />
     </material>
@@ -144,13 +144,12 @@
                 y="${chassis_big_width}"
                 z="${chassis_height}">
-                <!--TODO:Check  -->
                 <origin
-                    xyz="${chassis_total_length} ${chassis_big_width} ${chassis_height}"
-                    rpy="0 0 0" />` </xacro:inertial_box>
+                    xyz="0 0 ${chassis_height}"
+                    rpy="0 0 0" />
+            </xacro:inertial_box>
         </link>
     </xacro:macro>
     <!-- Chassis bottom !-->
-    <xacro:chassis
-        postfix="bottom" />
+    <xacro:chassis postfix="bottom" />
     <!-- Chassis mid !-->
     <xacro:chassis postfix="mid" />

File: model/description/ros2_control.xacro (robot description, xacro)
@@ -12,9 +12,9 @@
                 <param name="timeout_ms">1000</param>
                 <param name="loop_rate">30</param>
-                <param name="count_per_rev">20</param>
-                <param name="kp">100</param>
-                <param name="kd">30</param>
-                <param name="ki">10</param>
-                <param name="ko">100</param>
+                <param name="count_per_rev">823</param>
+                <param name="kp">12</param>
+                <param name="kd">0</param>
+                <param name="ki">5</param>
+                <param name="ko">50</param>
             </hardware>
             <joint name="left_front_wheel_joint">

File: model/description/wheels.xacro (robot description, xacro)
@@ -4,5 +4,5 @@
     <!-- |                                     Wheels                                      | -->
     <!-- =================================================================================== -->
-    <xacro:macro name="wheels" params="prefix">
+    <xacro:macro name="wheel" params="prefix">
         <link name="${prefix}_wheel">
             <visual>
@@ -25,13 +25,13 @@
         </link>
     </xacro:macro>
-    <xacro:wheels prefix="left_front" />
-    <xacro:wheels prefix="left_rear" />
-    <xacro:wheels prefix="right_front" />
-    <xacro:wheels prefix="right_rear" />
+    <xacro:wheel prefix="left_front" />
+    <xacro:wheel prefix="left_rear" />
+    <xacro:wheel prefix="right_front" />
+    <xacro:wheel prefix="right_rear" />
     <joint name="left_front_wheel_joint" type="continuous">
         <parent link="base_link" />
         <child link="left_front_wheel" />
         <origin
-            xyz="${chassis_big_length/2+(chassis_small_length+0.003)/2} ${chassis_small_width/2 + 0.015} 0.0"
+            xyz="${chassis_big_length/2+(chassis_small_length+0.003)/2} ${chassis_small_width/2 + wheel_thickness/2  + 0.015} 0.0"
             rpy="${-pi/2} 0.0 0.0" />
         <axis xyz="0 0 1" />
@@ -41,5 +41,5 @@
         <child link="left_rear_wheel" />
         <origin
-            xyz="-${chassis_big_length/2+(chassis_small_length+0.003)/2} ${chassis_small_width/2 + 0.015} 0.0"
+            xyz="-${chassis_big_length/2+(chassis_small_length+0.003)/2} ${chassis_small_width/2 + wheel_thickness/2+ 0.015} 0.0"
             rpy="${-pi/2} 0.0 0.0" />
         <axis xyz="0 0 1" />
@@ -49,5 +49,5 @@
         <child link="right_front_wheel" />
         <origin
-            xyz="${chassis_big_length/2+(chassis_small_length+0.003)/2} -${chassis_small_width/2 + 0.015} 0.0"
+            xyz="${chassis_big_length/2+(chassis_small_length+0.003)/2} -${chassis_small_width/2 + wheel_thickness/2+ 0.015} 0.0"
             rpy="${pi/2} 0.0 0.0" />
         <axis xyz="0 0 -1" />
@@ -57,5 +57,5 @@
         <child link="right_rear_wheel" />
         <origin
-            xyz="-${chassis_big_length/2+(chassis_small_length+0.003)/2} -${chassis_small_width/2 + 0.015} 0.0"
+            xyz="-${chassis_big_length/2+(chassis_small_length+0.003)/2} -${chassis_small_width/2 + wheel_thickness/2+ 0.015} 0.0"
             rpy="${pi/2} 0.0 0.0" />
         <axis xyz="0 0 -1" />

Commit message: Update model

File: model/description/others.xacro (robot description, xacro)
@@ -55,32 +55,4 @@
     </joint>
     <!-- =================================================================================== -->
-    <!-- |                                    Arduino                                      | -->
-    <!-- =================================================================================== -->
-    <!-- Raspberry -->
-    <link name="arduino">
-        <visual>
-            <geometry>
-                <box size="0.082 0.053 0.007" />
-            </geometry>
-            <origin xyz="0.0 0.0 0.0" rpy="0.0 0.0 0.0" />
-        </visual>
-        <collision>
-            <geometry>
-                <box size="0.082 0.053 0.007" />
-            </geometry>
-        </collision>
-        <xacro:inertial_box mass="0.080" x="0.082" y="0.053" z="0.007">
-            <origin xyz="0 0 0" rpy="0 0 0" />
-        </xacro:inertial_box>
-    </link>
-    <!-- Arduino joint-->
-    <joint name="arduino_joint" type="fixed">
-        <parent link="chassis_bottom" />
-        <child link="arduino" />
-        <origin
-            xyz="-${chassis_total_length/2 - 0.0265 - 0.03} ${chassis_small_width/2 - 0.041 - 0.015} ${0.0035 + chassis_height} "
-            rpy="0 0.0 ${pi/2}" />
-    </joint>
-    <!-- =================================================================================== -->
     <!-- |                                  Battery                                        | -->
     <!-- =================================================================================== -->
@@ -96,5 +68,5 @@
         <collision>
             <geometry>
-                <box size="0.071 0.065 0.035" />
+                <box size="0.075 0.065 0.035" />
             </geometry>
         </collision>
@@ -108,6 +80,6 @@
         <child link="battery" />
         <origin
-            xyz="-${chassis_total_length/2 - 0.0325 - 0.035} -${chassis_small_width/2 - 0.0375 - 0.015} ${0.0175 + chassis_height}"
-            rpy="0.0 0.0 ${pi/2}" />
+            xyz="-${chassis_total_length/2 - 0.0325 - 0.088} -${chassis_big_width/2 - 0.0375 - 0.083} ${0.0175 + chassis_height}"
+            rpy="0.0 0.0 0.0" />
     </joint>
     <!-- =================================================================================== -->
@@ -167,5 +139,5 @@
         <origin xyz="0 0 0" rpy="0.0 0.0 0.0" />
         <origin
-            xyz="${chassis_total_length/2 - 0.022 - 0.01} -${chassis_big_width/2 - 0.022- 0.05} 0.013"
+            xyz="${chassis_total_length/2 - 0.022 - 0.01} -${chassis_big_width/2 - 0.022- 0.071} 0.013"
             rpy="0.0 0.0
         0.0" />
@@ -197,6 +169,33 @@
         <child link="raspberry_pi" />
         <origin
-            xyz="${chassis_total_length/2 - 0.04745 -0.03} ${chassis_small_width/2 - 0.032 - 0.015} ${0.0125 + chassis_height}"
-            rpy="0.0 0.0 0.0" />
+            xyz="-${chassis_total_length/2 - 0.032 -0.015} ${chassis_small_width/2 - 0.04745 - 0.055} ${0.0125 + chassis_height}"
+            rpy="0.0 0.0 ${pi/2}" />
+    </joint>
+    <!-- =================================================================================== -->
+    <!-- |                                    Arduino                                      | -->
+    <!-- =================================================================================== -->
+    <link name="arduino">
+        <visual>
+            <geometry>
+                <box size="0.082 0.053 0.007" />
+            </geometry>
+            <origin xyz="0.0 0.0 0.0" rpy="0.0 0.0 0.0" />
+        </visual>
+        <collision>
+            <geometry>
+                <box size="0.082 0.053 0.007" />
+            </geometry>
+        </collision>
+        <xacro:inertial_box mass="0.080" x="0.082" y="0.053" z="0.007">
+            <origin xyz="0 0 0" rpy="0 0 0" />
+        </xacro:inertial_box>
+    </link>
+    <!-- Arduino joint-->
+    <joint name="arduino_joint" type="fixed">
+        <parent link="chassis_bottom" />
+        <child link="arduino" />
+        <origin
+            xyz="${chassis_total_length/2 - 0.041 - 0.001} ${chassis_big_width/2 - 0.0265 - 0.035} ${0.0035 + chassis_height} "
+            rpy="0 0.0 0.0" />
     </joint>
     <!-- =================================================================================== -->

File: model/description/robot_core.xacro (robot description, xacro)
@@ -45,5 +45,5 @@
     <xacro:property name="chassis_big_width" value="0.248" />
     <xacro:property name="chassis_height" value="0.004" />
-    <xacro:property name="chassis_mass" value="0.240" />
+    <xacro:property name="chassis_mass" value="0.150" />
     <xacro:property name="wheel_radius" value="0.033" />
     <xacro:property name="wheel_thickness" value="0.026" />

File: model/description/wheels.xacro (robot description, xacro)
@@ -33,5 +33,5 @@
         <child link="left_front_wheel" />
         <origin
-            xyz="${chassis_big_length/2+(chassis_small_length+0.003)/2} ${chassis_small_width/2 + wheel_thickness/2  + 0.015} 0.0"
+            xyz="${chassis_big_length/2+(chassis_small_length+0.003)/2} ${chassis_small_width/2 + wheel_thickness/2  + 0.005} 0.0"
             rpy="${-pi/2} 0.0 0.0" />
         <axis xyz="0 0 1" />
@@ -41,5 +41,5 @@
         <child link="left_rear_wheel" />
         <origin
-            xyz="-${chassis_big_length/2+(chassis_small_length+0.003)/2} ${chassis_small_width/2 + wheel_thickness/2+ 0.015} 0.0"
+            xyz="-${chassis_big_length/2+(chassis_small_length+0.003)/2} ${chassis_small_width/2 + wheel_thickness/2+ 0.005} 0.0"
             rpy="${-pi/2} 0.0 0.0" />
         <axis xyz="0 0 1" />
@@ -49,5 +49,5 @@
         <child link="right_front_wheel" />
         <origin
-            xyz="${chassis_big_length/2+(chassis_small_length+0.003)/2} -${chassis_small_width/2 + wheel_thickness/2+ 0.015} 0.0"
+            xyz="${chassis_big_length/2+(chassis_small_length+0.003)/2} -${chassis_small_width/2 + wheel_thickness/2+ 0.005} 0.0"
             rpy="${pi/2} 0.0 0.0" />
         <axis xyz="0 0 -1" />
@@ -57,5 +57,5 @@
         <child link="right_rear_wheel" />
         <origin
-            xyz="-${chassis_big_length/2+(chassis_small_length+0.003)/2} -${chassis_small_width/2 + wheel_thickness/2+ 0.015} 0.0"
+            xyz="-${chassis_big_length/2+(chassis_small_length+0.003)/2} -${chassis_small_width/2 + wheel_thickness/2+ 0.005} 0.0"
             rpy="${pi/2} 0.0 0.0" />
         <axis xyz="0 0 -1" />
